Commit message: 还差evaluate部分的整合,以及所有代码的测试. 发现由于torch版本不一样,计算结果好像不太一样

File: IsaacGymEnvs/assets/urdf/cartpolefull_temp.urdf (robot description, URDF)
Before this commit: robot cartpole_real_full, 3 links, 2 joints
Links:
- link pole: geometry collision box size=0.006 0.006 0.7855087679314434; visual box size=0.006 0.006 0.7855087679314434

Commit message: test done, need to add evaluate

File: IsaacGymEnvs/assets/urdf/cartpolefull_temp.urdf (robot description, URDF)
Before this commit: robot cartpole_real_full, 3 links, 2 joints
Links:
- link pole: geometry collision box size=0.006 0.006 0.5853582959985425; visual box size=0.006 0.006 0.5853582959985425

Commit message: test done, better README

File: IsaacGymEnvs/assets/urdf/cartpolefull_temp.urdf (robot description, URDF)
Before this commit: robot cartpole_real_full, 3 links, 2 joints
Links:
- link pole: geometry collision box size=0.006 0.006 0.3; visual box size=0.006 0.006 0.3
